File: kapukiTRX-hw-trx.sch (KiCad schematic (older format))
At the start: 25 parts, among them J1 GPS, J2 SWD, U1 STM32L476RGTx, U2 LP38693-3.3, Y1 16MHz

Commit message: Revert "Use it on mac"
This reverts commit 31182a4bd36aa13d038d509ee2b2cd4b0d770585.
Parts:
- C1, C10, C11, C2, C3, C4, C5, C6, C7, C8, C9: symbol kapukiTRX-hw-trx-rescue:C-Device -> Device:C
- D1: symbol kapukiTRX-hw-trx-rescue:LED_ARGB-Device -> Device:LED_ARGB
- D2: symbol kapukiTRX-hw-trx-rescue:LED-Device -> Device:LED
- FB1: symbol kapukiTRX-hw-trx-rescue:Ferrite_Bead-Device -> Device:Ferrite_Bead
- J1: symbol kapukiTRX-hw-trx-rescue:Conn_01x06-Connector_Generic -> Connector_Generic:Conn_01x06
- J2: symbol kapukiTRX-hw-trx-rescue:Conn_01x05-Connector_Generic -> Connector_Generic:Conn_01x05
- R1, R2, R3, R4, R5, R6: symbol kapukiTRX-hw-trx-rescue:R-Device -> Device:R
- U1: symbol kapukiTRX-hw-trx-rescue:STM32L476RGTx-MCU_ST_STM32L4 -> MCU_ST_STM32L4:STM32L476RGTx
- U2: symbol kapukiTRX-hw-trx-rescue:LP38693-LP38693 -> LP38693:LP38693
- Y1: symbol kapukiTRX-hw-trx-rescue:Crystal_GND24-Device -> Device:Crystal_GND24
Changed lines of the file:
@@
 $EndDescr
 $Comp
-L kapukiTRX-hw-trx-rescue:C-Device C4
+L Device:C C4
 U 1 1 5C749996
 P 1675 3150
@@
 $EndComp
 $Comp
-L kapukiTRX-hw-trx-rescue:C-Device C3
+L Device:C C3
 U 1 1 5C7499E6
 P 1675 2800
@@
 	1400 3150 1400 2800
 $Comp
-L kapukiTRX-hw-trx-rescue:C-Device C1
+L Device:C C1
 U 1 1 5C74B625
 P 1175 1100
@@
 $EndComp
 $Comp
-L kapukiTRX-hw-trx-rescue:C-Device C2
+L Device:C C2
 U 1 1 5C74B65F
 P 1625 1100
@@
 $EndComp
 $Comp
-L kapukiTRX-hw-trx-rescue:C-Device C6
+L Device:C C6
 U 1 1 5C74B691
 P 2100 1100
@@
 VCCCPU
 $Comp
-L kapukiTRX-hw-trx-rescue:C-Device C7
+L Device:C C7
 U 1 1 5C74E65D
 P 2640 1105
@@
 $EndComp
 $Comp
-L kapukiTRX-hw-trx-rescue:C-Device C8
+L Device:C C8
 U 1 1 5C74F6DB
 P 4200 1290
@@
 $EndComp
 $Comp
-L kapukiTRX-hw-trx-rescue:C-Device C9
+L Device:C C9
 U 1 1 5C74F723
 P 4600 1290
@@
 $EndComp
 $Comp
-L kapukiTRX-hw-trx-rescue:Ferrite_Bead-Device FB1
+L Device:Ferrite_Bead FB1
 U 1 1 5C74F867
 P 3825 925
@@
 RF1CLK
 $Comp
-L kapukiTRX-hw-trx-rescue:R-Device R4
+L Device:R R4
 U 1 1 5C7B6C85
 P 2350 2075
@@
 $EndSheet
 $Comp
-L kapukiTRX-hw-trx-rescue:LP38693-LP38693 U2
+L LP38693:LP38693 U2
 U 1 1 5C7DD5FC
 P 9625 1200
@@
 $EndComp
 $Comp
-L kapukiTRX-hw-trx-rescue:C-Device C11
+L Device:C C11
 U 1 1 5C7DD655
 P 10425 1250
@@
 $EndComp
 $Comp
-L kapukiTRX-hw-trx-rescue:C-Device C10
+L Device:C C10
 U 1 1 5C7DD6C5
 P 8475 1250
@@
 	8475 1000 8475 1100
 $Comp
-L kapukiTRX-hw-trx-rescue:R-Device R5
+L Device:R R5
 U 1 1 5C8015BC
 P 9025 1300
@@
 	5275 6855 5975 6855
 $Comp
-L kapukiTRX-hw-trx-rescue:Conn_01x06-Connector_Generic J1
+L Connector_Generic:Conn_01x06 J1
 U 1 1 5C9C8B95
 P 825 5725
@@
 GPSEN
 $Comp
-L kapukiTRX-hw-trx-rescue:Conn_01x05-Connector_Generic J2
+L Connector_Generic:Conn_01x05 J2
 U 1 1 5CC22AC7
 P 6175 6755
@@
 NRST
 $Comp
-L kapukiTRX-hw-trx-rescue:R-Device R6
+L Device:R R6
 U 1 1 5CC4355B
 P 10800 1275
@@
 $EndComp
 $Comp
-L kapukiTRX-hw-trx-rescue:LED-Device D2
+L Device:LED D2
 U 1 1 5CC43666
 P 10800 1750
@@
 	10800 1900 10800 1975
 $Comp
-L kapukiTRX-hw-trx-rescue:LED_ARGB-Device D1
+L Device:LED_ARGB D1
 U 1 1 5CC6499C
 P 1400 7175
@@
 $EndComp
 $Comp
-L kapukiTRX-hw-trx-rescue:R-Device R1
+L Device:R R1
 U 1 1 5CC64B2C
 P 1825 6975
@@
 $EndComp
 $Comp
-L kapukiTRX-hw-trx-rescue:R-Device R2
+L Device:R R2
 U 1 1 5CC64BCA
 P 1825 7175
@@
 $EndComp
 $Comp
-L kapukiTRX-hw-trx-rescue:R-Device R3
+L Device:R R3
 U 1 1 5CC64C2E
 P 1825 7375
@@
 	2375 2975 2350 2975
 $Comp
-L kapukiTRX-hw-trx-rescue:Crystal_GND24-Device Y1
+L Device:Crystal_GND24 Y1
 U 1 1 5CE6BFA7
 P 2150 2975
@@
 	2150 3150 2750 3150
 $Comp
-L kapukiTRX-hw-trx-rescue:C-Device C5
+L Device:C C5
 U 1 1 5CF3CB0A
 P 1950 2050
@@
 	4200 1465 4200 1440
 $Comp
-L kapukiTRX-hw-trx-rescue:STM32L476RGTx-MCU_ST_STM32L4 U1
+L MCU_ST_STM32L4:STM32L476RGTx U1
 U 1 1 5DB83729
 P 3625 3325

Commit message: Use it on mac
Parts:
- C1, C10, C11, C2, C3, C4, C5, C6, C7, C8, C9: symbol Device:C -> kapukiTRX-hw-trx-rescue:C-Device
- D1: symbol Device:LED_ARGB -> kapukiTRX-hw-trx-rescue:LED_ARGB-Device
- D2: symbol Device:LED -> kapukiTRX-hw-trx-rescue:LED-Device
- FB1: symbol Device:Ferrite_Bead -> kapukiTRX-hw-trx-rescue:Ferrite_Bead-Device
- J1: symbol Connector_Generic:Conn_01x06 -> kapukiTRX-hw-trx-rescue:Conn_01x06-Connector_Generic
- J2: symbol Connector_Generic:Conn_01x05 -> kapukiTRX-hw-trx-rescue:Conn_01x05-Connector_Generic
- R1, R2, R3, R4, R5, R6: symbol Device:R -> kapukiTRX-hw-trx-rescue:R-Device
- U1: symbol MCU_ST_STM32L4:STM32L476RGTx -> kapukiTRX-hw-trx-rescue:STM32L476RGTx-MCU_ST_STM32L4
- U2: symbol LP38693:LP38693 -> kapukiTRX-hw-trx-rescue:LP38693-LP38693
- Y1: symbol Device:Crystal_GND24 -> kapukiTRX-hw-trx-rescue:Crystal_GND24-Device
Changed lines of the file:
@@
 $EndDescr
 $Comp
-L Device:C C4
+L kapukiTRX-hw-trx-rescue:C-Device C4
 U 1 1 5C749996
 P 1675 3150
@@
 $EndComp
 $Comp
-L Device:C C3
+L kapukiTRX-hw-trx-rescue:C-Device C3
 U 1 1 5C7499E6
 P 1675 2800
@@
 	1400 3150 1400 2800
 $Comp
-L Device:C C1
+L kapukiTRX-hw-trx-rescue:C-Device C1
 U 1 1 5C74B625
 P 1175 1100
@@
 $EndComp
 $Comp
-L Device:C C2
+L kapukiTRX-hw-trx-rescue:C-Device C2
 U 1 1 5C74B65F
 P 1625 1100
@@
 $EndComp
 $Comp
-L Device:C C6
+L kapukiTRX-hw-trx-rescue:C-Device C6
 U 1 1 5C74B691
 P 2100 1100
@@
 VCCCPU
 $Comp
-L Device:C C7
+L kapukiTRX-hw-trx-rescue:C-Device C7
 U 1 1 5C74E65D
 P 2640 1105
@@
 $EndComp
 $Comp
-L Device:C C8
+L kapukiTRX-hw-trx-rescue:C-Device C8
 U 1 1 5C74F6DB
 P 4200 1290
@@
 $EndComp
 $Comp
-L Device:C C9
+L kapukiTRX-hw-trx-rescue:C-Device C9
 U 1 1 5C74F723
 P 4600 1290
@@
 $EndComp
 $Comp
-L Device:Ferrite_Bead FB1
+L kapukiTRX-hw-trx-rescue:Ferrite_Bead-Device FB1
 U 1 1 5C74F867
 P 3825 925
@@
 RF1CLK
 $Comp
-L Device:R R4
+L kapukiTRX-hw-trx-rescue:R-Device R4
 U 1 1 5C7B6C85
 P 2350 2075
@@
 $EndSheet
 $Comp
-L LP38693:LP38693 U2
+L kapukiTRX-hw-trx-rescue:LP38693-LP38693 U2
 U 1 1 5C7DD5FC
 P 9625 1200
@@
 $EndComp
 $Comp
-L Device:C C11
+L kapukiTRX-hw-trx-rescue:C-Device C11
 U 1 1 5C7DD655
 P 10425 1250
@@
 $EndComp
 $Comp
-L Device:C C10
+L kapukiTRX-hw-trx-rescue:C-Device C10
 U 1 1 5C7DD6C5
 P 8475 1250
@@
 	8475 1000 8475 1100
 $Comp
-L Device:R R5
+L kapukiTRX-hw-trx-rescue:R-Device R5
 U 1 1 5C8015BC
 P 9025 1300
@@
 	5275 6855 5975 6855
 $Comp
-L Connector_Generic:Conn_01x06 J1
+L kapukiTRX-hw-trx-rescue:Conn_01x06-Connector_Generic J1
 U 1 1 5C9C8B95
 P 825 5725
@@
 GPSEN
 $Comp
-L Connector_Generic:Conn_01x05 J2
+L kapukiTRX-hw-trx-rescue:Conn_01x05-Connector_Generic J2
 U 1 1 5CC22AC7
 P 6175 6755
@@
 NRST
 $Comp
-L Device:R R6
+L kapukiTRX-hw-trx-rescue:R-Device R6
 U 1 1 5CC4355B
 P 10800 1275
@@
 $EndComp
 $Comp
-L Device:LED D2
+L kapukiTRX-hw-trx-rescue:LED-Device D2
 U 1 1 5CC43666
 P 10800 1750
@@
 	10800 1900 10800 1975
 $Comp
-L Device:LED_ARGB D1
+L kapukiTRX-hw-trx-rescue:LED_ARGB-Device D1
 U 1 1 5CC6499C
 P 1400 7175
@@
 $EndComp
 $Comp
-L Device:R R1
+L kapukiTRX-hw-trx-rescue:R-Device R1
 U 1 1 5CC64B2C
 P 1825 6975
@@
 $EndComp
 $Comp
-L Device:R R2
+L kapukiTRX-hw-trx-rescue:R-Device R2
 U 1 1 5CC64BCA
 P 1825 7175
@@
 $EndComp
 $Comp
-L Device:R R3
+L kapukiTRX-hw-trx-rescue:R-Device R3
 U 1 1 5CC64C2E
 P 1825 7375
@@
 	2375 2975 2350 2975
 $Comp
-L Device:Crystal_GND24 Y1
+L kapukiTRX-hw-trx-rescue:Crystal_GND24-Device Y1
 U 1 1 5CE6BFA7
 P 2150 2975
@@
 	2150 3150 2750 3150
 $Comp
-L Device:C C5
+L kapukiTRX-hw-trx-rescue:C-Device C5
 U 1 1 5CF3CB0A
 P 1950 2050
@@
 	4200 1465 4200 1440
 $Comp
-L MCU_ST_STM32L4:STM32L476RGTx U1
+L kapukiTRX-hw-trx-rescue:STM32L476RGTx-MCU_ST_STM32L4 U1
 U 1 1 5DB83729
 P 3625 3325
