File: rfmodules.sch (KiCad schematic (older format))
At the start: 8 parts, among them U6 LP38693SD-3.3

Commit message: Revert "Use it on mac"
This reverts commit 31182a4bd36aa13d038d509ee2b2cd4b0d770585.
Parts:
- A1, A2: symbol kapukiTRX-hw-trx-rescue:E28-2G4M20S-SX1280 -> SX1280:E28-2G4M20S
- C28, C29, C31, C32: symbol kapukiTRX-hw-trx-rescue:C-Device -> Device:C
- C30: symbol kapukiTRX-hw-trx-rescue:CP-Device -> Device:CP
- U6: symbol kapukiTRX-hw-trx-rescue:LP38693-LP38693 -> LP38693:LP38693
Changed lines of the file:
@@
 $EndComp
 $Comp
-L kapukiTRX-hw-trx-rescue:LP38693-LP38693 U6
+L LP38693:LP38693 U6
 U 1 1 5C7BA578
 P 2500 1925
@@
 $EndComp
 $Comp
-L kapukiTRX-hw-trx-rescue:C-Device C29
+L Device:C C29
 U 1 1 5C7BA5D5
 P 3125 1975
@@
 $EndComp
 $Comp
-L kapukiTRX-hw-trx-rescue:C-Device C28
+L Device:C C28
 U 1 1 5C7BA627
 P 1675 1975
@@
 Connection ~ 1675 2250
 $Comp
-L kapukiTRX-hw-trx-rescue:C-Device C31
+L Device:C C31
 U 1 1 5C7CD227
 P 4375 1825
@@
 $EndComp
 $Comp
-L kapukiTRX-hw-trx-rescue:C-Device C32
+L Device:C C32
 U 1 1 5C7CD2B2
 P 4375 4350
@@
 	4075 4350 4075 4725
 $Comp
-L kapukiTRX-hw-trx-rescue:CP-Device C30
+L Device:CP C30
 U 1 1 5C8A056F
 P 3725 2025
@@
 	3725 2225 3725 2175
 $Comp
-L kapukiTRX-hw-trx-rescue:E28-2G4M20S-SX1280 A1
+L SX1280:E28-2G4M20S A1
 U 1 1 5C8B677C
 P 4075 5275
@@
 $EndComp
 $Comp
-L kapukiTRX-hw-trx-rescue:E28-2G4M20S-SX1280 A2
+L SX1280:E28-2G4M20S A2
 U 1 1 5C8B6803
 P 4100 3000

Commit message: Use it on mac
Parts:
- A1, A2: symbol SX1280:E28-2G4M20S -> kapukiTRX-hw-trx-rescue:E28-2G4M20S-SX1280
- C28, C29, C31, C32: symbol Device:C -> kapukiTRX-hw-trx-rescue:C-Device
- C30: symbol Device:CP -> kapukiTRX-hw-trx-rescue:CP-Device
- U6: symbol LP38693:LP38693 -> kapukiTRX-hw-trx-rescue:LP38693-LP38693
Changed lines of the file:
@@
 $EndComp
 $Comp
-L LP38693:LP38693 U6
+L kapukiTRX-hw-trx-rescue:LP38693-LP38693 U6
 U 1 1 5C7BA578
 P 2500 1925
@@
 $EndComp
 $Comp
-L Device:C C29
+L kapukiTRX-hw-trx-rescue:C-Device C29
 U 1 1 5C7BA5D5
 P 3125 1975
@@
 $EndComp
 $Comp
-L Device:C C28
+L kapukiTRX-hw-trx-rescue:C-Device C28
 U 1 1 5C7BA627
 P 1675 1975
@@
 Connection ~ 1675 2250
 $Comp
-L Device:C C31
+L kapukiTRX-hw-trx-rescue:C-Device C31
 U 1 1 5C7CD227
 P 4375 1825
@@
 $EndComp
 $Comp
-L Device:C C32
+L kapukiTRX-hw-trx-rescue:C-Device C32
 U 1 1 5C7CD2B2
 P 4375 4350
@@
 	4075 4350 4075 4725
 $Comp
-L Device:CP C30
+L kapukiTRX-hw-trx-rescue:CP-Device C30
 U 1 1 5C8A056F
 P 3725 2025
@@
 	3725 2225 3725 2175
 $Comp
-L SX1280:E28-2G4M20S A1
+L kapukiTRX-hw-trx-rescue:E28-2G4M20S-SX1280 A1
 U 1 1 5C8B677C
 P 4075 5275
@@
 $EndComp
 $Comp
-L SX1280:E28-2G4M20S A2
+L kapukiTRX-hw-trx-rescue:E28-2G4M20S-SX1280 A2
 U 1 1 5C8B6803
 P 4100 3000
