File: rfmodules.sch (KiCad schematic (older format))
At the start: 8 parts, among them U6 LP38693SD-3.3

Commit message: Final changes for rev.3
Other:
- note added: "RF1 module"
- note added: "RF2 module"
- moved on the sheet: A1, A2, C28, C29, C30, C31, C32, U6

Commit message: Make some value changes for consistency
Parts:
- U6: value LP38693SD-3.3 -> LP38693-3.3
Changed lines of the file:
@@
 EESchema Schematic File Version 4
-LIBS:kapukiTRX-hw-trx-cache
 EELAYER 30 0
 EELAYER END
@@
 P 4050 1925
 F 0 "U6" H 4050 2290 50  0000 C CNN
-F 1 "LP38693SD-3.3" H 4050 2199 50  0000 C CNN
+F 1 "LP38693-3.3" H 4050 2199 50  0000 C CNN
 F 2 "miscellaneous:WSON-6_3x3mm_Pitch0.95mm" H 4050 1925 50  0001 C CNN
 F 3 "http://www.ti.com/lit/ds/snvs321o/snvs321o.pdf" H 4050 1925 50  0001 C CNN
