File: connectors.sch (KiCad schematic (older format))
At the start: 40 parts, among them J10 Conn_01x01, J11 Conn_01x01, J12 Conn_01x01, J13 Conn_01x01, J14 Conn_01x01, J15 Conn_01x01, J16 Conn_01x01, J17 Conn_01x01, J18 Conn_01x01, J19 GND for the Servo connectors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

Commit message: Use it on mac
Parts:
- C12, C13, C14, C15, C16, C17, C18, C19, C20, C21, C23, C24, C25, C26: symbol Device:C -> kapukiTRX-hw-trx-rescue:C-Device
- C22, C27: symbol Device:CP -> kapukiTRX-hw-trx-rescue:CP-Device
- J10, J11, J12, J13, J14, J15, J16, J17, J18, J19, J3, J4, J5, J6, J7, J8, J9: symbol Connector_Generic:Conn_01x01 -> kapukiTRX-hw-trx-rescue:Conn_01x01-Connector_Generic
- J20: symbol Connector_Generic:Conn_01x03 -> kapukiTRX-hw-trx-rescue:Conn_01x03-Connector_Generic
- R7, R8, R9: symbol Device:R -> kapukiTRX-hw-trx-rescue:R-Device
- U3: symbol dk_Logic-Translators-Level-Shifters:TXB0108PWR -> kapukiTRX-hw-trx-rescue:TXB0108PWR-dk_Logic-Translators-Level-Shifters
- U4: symbol LP38693:LP38693 -> kapukiTRX-hw-trx-rescue:LP38693-LP38693
- U5: symbol Interface_CAN_LIN:MCP2562-E-MF -> kapukiTRX-hw-trx-rescue:MCP2562-E-MF-Interface_CAN_LIN
Changed lines of the file:
@@
 	8375 2150 8225 2150
 $Comp
-L Device:C C23
+L kapukiTRX-hw-trx-rescue:C-Device C23
 U 1 1 5C78CA1B
 P 6550 2250
@@
 $EndComp
 $Comp
-L Device:C C25
+L kapukiTRX-hw-trx-rescue:C-Device C25
 U 1 1 5C78CA91
 P 8375 2300
@@
 	2925 3400 3200 3400
 $Comp
-L Device:CP C22
+L kapukiTRX-hw-trx-rescue:CP-Device C22
 U 1 1 5C79ED78
 P 6100 2250
@@
 	6100 2500 6550 2500
 $Comp
-L LP38693:LP38693 U4
+L kapukiTRX-hw-trx-rescue:LP38693-LP38693 U4
 U 1 1 5C7B161D
 P 7825 2150
@@
 $EndComp
 $Comp
-L Device:C C13
+L kapukiTRX-hw-trx-rescue:C-Device C13
 U 1 1 5C7D119D
 P 3950 2900
@@
 	4175 2900 4175 2950
 $Comp
-L Device:C C12
+L kapukiTRX-hw-trx-rescue:C-Device C12
 U 1 1 5C7D7B7F
 P 3300 2900
@@
 	8370 3855 8370 3705
 $Comp
-L Device:C C?
+L kapukiTRX-hw-trx-rescue:C-Device C?
 U 1 1 5CCDDFB0
 P 8595 3705
@@
 	8370 3705 8370 3555
 $Comp
-L Device:R R?
+L kapukiTRX-hw-trx-rescue:R-Device R?
 U 1 1 5CCDDFD0
 P 9320 4655
@@
 Connection ~ 9320 4355
 $Comp
-L Connector_Generic:Conn_01x03 J?
+L kapukiTRX-hw-trx-rescue:Conn_01x03-Connector_Generic J?
 U 1 1 5CCDDFDF
 P 10245 4355
@@
 	9945 4455 10045 4455
 $Comp
-L Device:C C19
+L kapukiTRX-hw-trx-rescue:C-Device C19
 U 1 1 5CCE1675
 P 4700 2950
@@
 $EndComp
 $Comp
-L Device:C C18
+L kapukiTRX-hw-trx-rescue:C-Device C18
 U 1 1 5CCE1727
 P 4700 2500
@@
 	4700 2350 5250 2350
 $Comp
-L Device:C C14
+L kapukiTRX-hw-trx-rescue:C-Device C14
 U 1 1 5CCE1785
 P 4200 5700
@@
 $EndComp
 $Comp
-L Device:C C15
+L kapukiTRX-hw-trx-rescue:C-Device C15
 U 1 1 5CCE1C56
 P 4350 5250
@@
 $EndComp
 $Comp
-L Device:C C16
+L kapukiTRX-hw-trx-rescue:C-Device C16
 U 1 1 5CCE1CA6
 P 4500 4800
@@
 $EndComp
 $Comp
-L Device:C C17
+L kapukiTRX-hw-trx-rescue:C-Device C17
 U 1 1 5CCE1CFA
 P 4650 4350
@@
 Connection ~ 4650 4150
 $Comp
-L Device:C C21
+L kapukiTRX-hw-trx-rescue:C-Device C21
 U 1 1 5CD045AA
 P 4775 3925
@@
 $EndComp
 $Comp
-L Device:C C20
+L kapukiTRX-hw-trx-rescue:C-Device C20
 U 1 1 5CD17DAF
 P 4700 3400
@@
 	4700 3250 5250 3250
 $Comp
-L Device:R R8
+L kapukiTRX-hw-trx-rescue:R-Device R8
 U 1 1 5CD7AFCF
 P 7200 2250
@@
 CANTX
 $Comp
-L Device:CP C27
+L kapukiTRX-hw-trx-rescue:CP-Device C27
 U 1 1 5CE22492
 P 8750 2300
@@
 VCC
 $Comp
-L Connector_Generic:Conn_01x01 J19
+L kapukiTRX-hw-trx-rescue:Conn_01x01-Connector_Generic J19
 U 1 1 5CF3538C
 P 5450 6350
@@
 	5200 6350 5250 6350
 $Comp
-L dk_Logic-Translators-Level-Shifters:TXB0108PWR U3
+L kapukiTRX-hw-trx-rescue:TXB0108PWR-dk_Logic-Translators-Level-Shifters U3
 U 1 1 5CB75ACC
 P 3600 3700
@@
 	3900 3700 4775 3700
 $Comp
-L Device:R R7
+L kapukiTRX-hw-trx-rescue:R-Device R7
 U 1 1 5CBE1CAD
 P 3150 4400
@@
 	8370 4690 8370 4655
 $Comp
-L Connector_Generic:Conn_01x01 J5
+L kapukiTRX-hw-trx-rescue:Conn_01x01-Connector_Generic J5
 U 1 1 5DD3888B
 P 5450 2800
@@
 $EndComp
 $Comp
-L Connector_Generic:Conn_01x01 J6
+L kapukiTRX-hw-trx-rescue:Conn_01x01-Connector_Generic J6
 U 1 1 5DD38C93
 P 5450 2900
@@
 $EndComp
 $Comp
-L Connector_Generic:Conn_01x01 J7
+L kapukiTRX-hw-trx-rescue:Conn_01x01-Connector_Generic J7
 U 1 1 5DD38FAD
 P 5450 3250
@@
 $EndComp
 $Comp
-L Connector_Generic:Conn_01x01 J8
+L kapukiTRX-hw-trx-rescue:Conn_01x01-Connector_Generic J8
 U 1 1 5DD39454
 P 5450 3350
@@
 $EndComp
 $Comp
-L Connector_Generic:Conn_01x01 J9
+L kapukiTRX-hw-trx-rescue:Conn_01x01-Connector_Generic J9
 U 1 1 5DD3999D
 P 5450 3700
@@
 $EndComp
 $Comp
-L Connector_Generic:Conn_01x01 J10
+L kapukiTRX-hw-trx-rescue:Conn_01x01-Connector_Generic J10
 U 1 1 5DD39E93
 P 5450 3800
@@
 $EndComp
 $Comp
-L Connector_Generic:Conn_01x01 J11
+L kapukiTRX-hw-trx-rescue:Conn_01x01-Connector_Generic J11
 U 1 1 5DD3A2CD
 P 5450 4150
@@
 $EndComp
 $Comp
-L Connector_Generic:Conn_01x01 J12
+L kapukiTRX-hw-trx-rescue:Conn_01x01-Connector_Generic J12
 U 1 1 5DD3A7A0
 P 5450 4250
@@
 $EndComp
 $Comp
-L Connector_Generic:Conn_01x01 J13
+L kapukiTRX-hw-trx-rescue:Conn_01x01-Connector_Generic J13
 U 1 1 5DD3AC57
 P 5450 4600
@@
 $EndComp
 $Comp
-L Connector_Generic:Conn_01x01 J14
+L kapukiTRX-hw-trx-rescue:Conn_01x01-Connector_Generic J14
 U 1 1 5DD3B03C
 P 5450 4700
@@
 $EndComp
 $Comp
-L Connector_Generic:Conn_01x01 J15
+L kapukiTRX-hw-trx-rescue:Conn_01x01-Connector_Generic J15
 U 1 1 5DD3B325
 P 5450 5050
@@
 $EndComp
 $Comp
-L Connector_Generic:Conn_01x01 J16
+L kapukiTRX-hw-trx-rescue:Conn_01x01-Connector_Generic J16
 U 1 1 5DD3B787
 P 5450 5150
@@
 $EndComp
 $Comp
-L Connector_Generic:Conn_01x01 J17
+L kapukiTRX-hw-trx-rescue:Conn_01x01-Connector_Generic J17
 U 1 1 5DD3BAAC
 P 5450 5500
@@
 $EndComp
 $Comp
-L Connector_Generic:Conn_01x01 J18
+L kapukiTRX-hw-trx-rescue:Conn_01x01-Connector_Generic J18
 U 1 1 5DD3C08C
 P 5450 5600
@@
 $EndComp
 $Comp
-L Interface_CAN_LIN:MCP2562-E-MF U5
+L kapukiTRX-hw-trx-rescue:MCP2562-E-MF-Interface_CAN_LIN U5
 U 1 1 5DC41DB4
 P 8370 4255
@@
 	7625 4455 7870 4455
 $Comp
-L Device:C C?
+L kapukiTRX-hw-trx-rescue:C-Device C?
 U 1 1 5DC9B7C0
 P 7755 4725
@@
 	7755 4355 7870 4355
 $Comp
-L Connector_Generic:Conn_01x01 J4
+L kapukiTRX-hw-trx-rescue:Conn_01x01-Connector_Generic J4
 U 1 1 5DD384FB
 P 5450 2450
@@
 $EndComp
 $Comp
-L Connector_Generic:Conn_01x01 J3
+L kapukiTRX-hw-trx-rescue:Conn_01x01-Connector_Generic J3
 U 1 1 5DD37C43
 P 5450 2350

Commit message: Revert "Use it on mac"
This reverts commit 31182a4bd36aa13d038d509ee2b2cd4b0d770585.
Parts:
- C12, C13, C14, C15, C16, C17, C18, C19, C20, C21, C23, C24, C25, C26: symbol kapukiTRX-hw-trx-rescue:C-Device -> Device:C
- C22, C27: symbol kapukiTRX-hw-trx-rescue:CP-Device -> Device:CP
- J10, J11, J12, J13, J14, J15, J16, J17, J18, J19, J3, J4, J5, J6, J7, J8, J9: symbol kapukiTRX-hw-trx-rescue:Conn_01x01-Connector_Generic -> Connector_Generic:Conn_01x01
- J20: symbol kapukiTRX-hw-trx-rescue:Conn_01x03-Connector_Generic -> Connector_Generic:Conn_01x03
- R7, R8, R9: symbol kapukiTRX-hw-trx-rescue:R-Device -> Device:R
- U3: symbol kapukiTRX-hw-trx-rescue:TXB0108PWR-dk_Logic-Translators-Level-Shifters -> dk_Logic-Translators-Level-Shifters:TXB0108PWR
- U4: symbol kapukiTRX-hw-trx-rescue:LP38693-LP38693 -> LP38693:LP38693
- U5: symbol kapukiTRX-hw-trx-rescue:MCP2562-E-MF-Interface_CAN_LIN -> Interface_CAN_LIN:MCP2562-E-MF
Changed lines of the file:
@@
 	8375 2150 8225 2150
 $Comp
-L kapukiTRX-hw-trx-rescue:C-Device C23
+L Device:C C23
 U 1 1 5C78CA1B
 P 6550 2250
@@
 $EndComp
 $Comp
-L kapukiTRX-hw-trx-rescue:C-Device C25
+L Device:C C25
 U 1 1 5C78CA91
 P 8375 2300
@@
 	2925 3400 3200 3400
 $Comp
-L kapukiTRX-hw-trx-rescue:CP-Device C22
+L Device:CP C22
 U 1 1 5C79ED78
 P 6100 2250
@@
 	6100 2500 6550 2500
 $Comp
-L kapukiTRX-hw-trx-rescue:LP38693-LP38693 U4
+L LP38693:LP38693 U4
 U 1 1 5C7B161D
 P 7825 2150
@@
 $EndComp
 $Comp
-L kapukiTRX-hw-trx-rescue:C-Device C13
+L Device:C C13
 U 1 1 5C7D119D
 P 3950 2900
@@
 	4175 2900 4175 2950
 $Comp
-L kapukiTRX-hw-trx-rescue:C-Device C12
+L Device:C C12
 U 1 1 5C7D7B7F
 P 3300 2900
@@
 	8370 3855 8370 3705
 $Comp
-L kapukiTRX-hw-trx-rescue:C-Device C?
+L Device:C C?
 U 1 1 5CCDDFB0
 P 8595 3705
@@
 	8370 3705 8370 3555
 $Comp
-L kapukiTRX-hw-trx-rescue:R-Device R?
+L Device:R R?
 U 1 1 5CCDDFD0
 P 9320 4655
@@
 Connection ~ 9320 4355
 $Comp
-L kapukiTRX-hw-trx-rescue:Conn_01x03-Connector_Generic J?
+L Connector_Generic:Conn_01x03 J?
 U 1 1 5CCDDFDF
 P 10245 4355
@@
 	9945 4455 10045 4455
 $Comp
-L kapukiTRX-hw-trx-rescue:C-Device C19
+L Device:C C19
 U 1 1 5CCE1675
 P 4700 2950
@@
 $EndComp
 $Comp
-L kapukiTRX-hw-trx-rescue:C-Device C18
+L Device:C C18
 U 1 1 5CCE1727
 P 4700 2500
@@
 	4700 2350 5250 2350
 $Comp
-L kapukiTRX-hw-trx-rescue:C-Device C14
+L Device:C C14
 U 1 1 5CCE1785
 P 4200 5700
@@
 $EndComp
 $Comp
-L kapukiTRX-hw-trx-rescue:C-Device C15
+L Device:C C15
 U 1 1 5CCE1C56
 P 4350 5250
@@
 $EndComp
 $Comp
-L kapukiTRX-hw-trx-rescue:C-Device C16
+L Device:C C16
 U 1 1 5CCE1CA6
 P 4500 4800
@@
 $EndComp
 $Comp
-L kapukiTRX-hw-trx-rescue:C-Device C17
+L Device:C C17
 U 1 1 5CCE1CFA
 P 4650 4350
@@
 Connection ~ 4650 4150
 $Comp
-L kapukiTRX-hw-trx-rescue:C-Device C21
+L Device:C C21
 U 1 1 5CD045AA
 P 4775 3925
@@
 $EndComp
 $Comp
-L kapukiTRX-hw-trx-rescue:C-Device C20
+L Device:C C20
 U 1 1 5CD17DAF
 P 4700 3400
@@
 	4700 3250 5250 3250
 $Comp
-L kapukiTRX-hw-trx-rescue:R-Device R8
+L Device:R R8
 U 1 1 5CD7AFCF
 P 7200 2250
@@
 CANTX
 $Comp
-L kapukiTRX-hw-trx-rescue:CP-Device C27
+L Device:CP C27
 U 1 1 5CE22492
 P 8750 2300
@@
 VCC
 $Comp
-L kapukiTRX-hw-trx-rescue:Conn_01x01-Connector_Generic J19
+L Connector_Generic:Conn_01x01 J19
 U 1 1 5CF3538C
 P 5450 6350
@@
 	5200 6350 5250 6350
 $Comp
-L kapukiTRX-hw-trx-rescue:TXB0108PWR-dk_Logic-Translators-Level-Shifters U3
+L dk_Logic-Translators-Level-Shifters:TXB0108PWR U3
 U 1 1 5CB75ACC
 P 3600 3700
@@
 	3900 3700 4775 3700
 $Comp
-L kapukiTRX-hw-trx-rescue:R-Device R7
+L Device:R R7
 U 1 1 5CBE1CAD
 P 3150 4400
@@
 	8370 4690 8370 4655
 $Comp
-L kapukiTRX-hw-trx-rescue:Conn_01x01-Connector_Generic J5
+L Connector_Generic:Conn_01x01 J5
 U 1 1 5DD3888B
 P 5450 2800
@@
 $EndComp
 $Comp
-L kapukiTRX-hw-trx-rescue:Conn_01x01-Connector_Generic J6
+L Connector_Generic:Conn_01x01 J6
 U 1 1 5DD38C93
 P 5450 2900
@@
 $EndComp
 $Comp
-L kapukiTRX-hw-trx-rescue:Conn_01x01-Connector_Generic J7
+L Connector_Generic:Conn_01x01 J7
 U 1 1 5DD38FAD
 P 5450 3250
@@
 $EndComp
 $Comp
-L kapukiTRX-hw-trx-rescue:Conn_01x01-Connector_Generic J8
+L Connector_Generic:Conn_01x01 J8
 U 1 1 5DD39454
 P 5450 3350
@@
 $EndComp
 $Comp
-L kapukiTRX-hw-trx-rescue:Conn_01x01-Connector_Generic J9
+L Connector_Generic:Conn_01x01 J9
 U 1 1 5DD3999D
 P 5450 3700
@@
 $EndComp
 $Comp
-L kapukiTRX-hw-trx-rescue:Conn_01x01-Connector_Generic J10
+L Connector_Generic:Conn_01x01 J10
 U 1 1 5DD39E93
 P 5450 3800
@@
 $EndComp
 $Comp
-L kapukiTRX-hw-trx-rescue:Conn_01x01-Connector_Generic J11
+L Connector_Generic:Conn_01x01 J11
 U 1 1 5DD3A2CD
 P 5450 4150
@@
 $EndComp
 $Comp
-L kapukiTRX-hw-trx-rescue:Conn_01x01-Connector_Generic J12
+L Connector_Generic:Conn_01x01 J12
 U 1 1 5DD3A7A0
 P 5450 4250
@@
 $EndComp
 $Comp
-L kapukiTRX-hw-trx-rescue:Conn_01x01-Connector_Generic J13
+L Connector_Generic:Conn_01x01 J13
 U 1 1 5DD3AC57
 P 5450 4600
@@
 $EndComp
 $Comp
-L kapukiTRX-hw-trx-rescue:Conn_01x01-Connector_Generic J14
+L Connector_Generic:Conn_01x01 J14
 U 1 1 5DD3B03C
 P 5450 4700
@@
 $EndComp
 $Comp
-L kapukiTRX-hw-trx-rescue:Conn_01x01-Connector_Generic J15
+L Connector_Generic:Conn_01x01 J15
 U 1 1 5DD3B325
 P 5450 5050
@@
 $EndComp
 $Comp
-L kapukiTRX-hw-trx-rescue:Conn_01x01-Connector_Generic J16
+L Connector_Generic:Conn_01x01 J16
 U 1 1 5DD3B787
 P 5450 5150
@@
 $EndComp
 $Comp
-L kapukiTRX-hw-trx-rescue:Conn_01x01-Connector_Generic J17
+L Connector_Generic:Conn_01x01 J17
 U 1 1 5DD3BAAC
 P 5450 5500
@@
 $EndComp
 $Comp
-L kapukiTRX-hw-trx-rescue:Conn_01x01-Connector_Generic J18
+L Connector_Generic:Conn_01x01 J18
 U 1 1 5DD3C08C
 P 5450 5600
@@
 $EndComp
 $Comp
-L kapukiTRX-hw-trx-rescue:MCP2562-E-MF-Interface_CAN_LIN U5
+L Interface_CAN_LIN:MCP2562-E-MF U5
 U 1 1 5DC41DB4
 P 8370 4255
@@
 	7625 4455 7870 4455
 $Comp
-L kapukiTRX-hw-trx-rescue:C-Device C?
+L Device:C C?
 U 1 1 5DC9B7C0
 P 7755 4725
@@
 	7755 4355 7870 4355
 $Comp
-L kapukiTRX-hw-trx-rescue:Conn_01x01-Connector_Generic J4
+L Connector_Generic:Conn_01x01 J4
 U 1 1 5DD384FB
 P 5450 2450
@@
 $EndComp
 $Comp
-L kapukiTRX-hw-trx-rescue:Conn_01x01-Connector_Generic J3
+L Connector_Generic:Conn_01x01 J3
 U 1 1 5DD37C43
 P 5450 2350
