File: sensors.sch (KiCad schematic (older format))
At the start: 14 parts

Commit message: Wiring sensors
Parts:
- removed R? (x2): 4k7, symbol Device:R
- removed R?: R, symbol Device:R
- added C33, C34: 100n, Capacitor_SMD:C_0402_1005Metric, symbol Device:C
- added C35: 6n8, Capacitor_SMD:C_0402_1005Metric, symbol Device:C
- added R13: 10k, Resistor_SMD:R_0402_1005Metric, symbol Device:R
- C36: renamed from C?; value 100n -> 120n; footprint (none) -> Capacitor_SMD:C_0402_1005Metric
- C37, C38, C39, C40: renamed from C?; footprint (none) -> Capacitor_SMD:C_0402_1005Metric
- R10, R11: renamed from R?; footprint (none) -> Resistor_SMD:R_0402_1005Metric
- R12: renamed from R?; value 4k7 -> 10k; footprint (none) -> Resistor_SMD:R_0402_1005Metric
- Y2: renamed from Y?; value Crystal -> 32.768kHz; footprint (none) -> Crystal:Crystal_SMD_3215-2Pin_3.2x1.5mm
- gave numbers to parts that had none: 2
Connections:
- net VCCCPU is gone; now on net VCC: C36.2, C37.2, R10.1, R11.1, R12.1, U7.28 (VDDIO), U7.3 (VDD), U8.1 (VDDIO), U8.10 (VCC)
- net GND: now also U7.17 (COM3), U7.5 (PS1), U7.6 (PS0), U8.3 (GND), U8.9 (GND), C33.2, C34.2, C35.1
- net BNORESET: now reaches U7.11 (~nRESET)
- net BNORESET: now also R13.2
- net BNOINT: now reaches U7.14 (INT)
- net VCC: now reaches U8.5 (SDO)
- net VCC: now also U8.6 (CSB), C33.1, C34.1, C35.2, R13.1
- net BMPINT: now reaches U8.7 (INT)
- net SCA renamed SDA
- no-connect marks 0 -> 1
Other:
- moved on the sheet: R10, R11, R12

Commit message: Use crystal with smaller footprint
Parts:
- Y2: footprint Crystal:Crystal_SMD_3215-2Pin_3.2x1.5mm -> Crystal:Crystal_SMD_2012-2Pin_2.0x1.2mm
Changed lines of the file:
@@
 F 0 "Y2" V 5354 2681 50  0000 L CNN
 F 1 "32.768kHz" V 5445 2681 50  0000 L CNN
-F 2 "Crystal:Crystal_SMD_3215-2Pin_3.2x1.5mm" H 5400 2550 50  0001 C CNN
+F 2 "Crystal:Crystal_SMD_2012-2Pin_2.0x1.2mm" H 5400 2550 50  0001 C CNN
 F 3 "~" H 5400 2550 50  0001 C CNN
 	1    5400 2550

Commit message: Add proper footprint for BMP388
Parts:
- U8: footprint (none) -> miscellaneous:Bosch_LGA10_2x2mm_Pitch0.5mm
Changed lines of the file:
@@
 F 0 "U8" H 4350 6300 50  0000 L CNN
 F 1 "BMP388" H 4750 6300 50  0000 L CNN
-F 2 "" H 4650 5850 50  0001 C CNN
-F 3 "" H 4650 5850 50  0001 C CNN
+F 2 "miscellaneous:Bosch_LGA10_2x2mm_Pitch0.5mm" H 4650 5850 50  0001 C CNN
+F 3 "https://www.mouser.com/pdfdocs/BST-BMP388-DS001-01.pdf" H 4650 5850 50  0001 C CNN
 	1    4650 5850
 	1    0    0    -1
